File: PCB/pico/voltex_pico.kicad_sch (KiCad schematic)
At the start: 63 parts, among them U1 PiPico, U2 ADG708BRUZ, U3 TMAG5273, U4 TMAG5273, U5 DC/DC

Commit message: PCB progress 70%
Parts:
- removed JA1, JA2, JB1, JB2: Conn_01x04, voltex_pico:SH1.0_4P_Solder_Combo, symbol Connector_Generic:Conn_01x04
- added C11, C12, C13, C14, C15, C16: 0.1uF, Capacitor_SMD:C_0603_1608Metric_Pad1.08x0.95mm_HandSolder, symbol Device:C
- added DL1, DL2, DL3, DL4, DL5, DL6, DR1, DR2, DR3, DR4, DR5, DR6: WS2812B_Unified, voltex_pico:WS2812B-4020, symbol voltex_pico:WS2812B_Unified
- added J1, J2, J3, J4: Conn_01x06_Socket, voltex_pico:Solder_6P, symbol Connector:Conn_01x06_Socket
- renumbered C26 to C10, C10 to C8, C11 to C9
Connections:
- net VB1 is gone; now on net V1: C8.1
- net +3V3: now also J1.1 (Pin_1), J2.1 (Pin_1), J3.1 (Pin_1), J4.1 (Pin_1)
- net +5V: now also C11.1, C12.1, C13.1, C14.1, C15.1, C16.1, DL1.V (VDD), DL2.V (VDD), DL3.V (VDD), DL4.V (VDD), DL5.V (VDD), DL6.V (VDD), DR1.V (VDD), DR2.V (VDD), DR3.V (VDD), DR4.V (VDD), DR5.V (VDD), DR6.V (VDD), J1.5 (Pin_5), J2.5 (Pin_5), J3.5 (Pin_5), J4.5 (Pin_5)
- net GND: now also C11.2, C12.2, C13.2, C14.2, C15.2, C16.2, DL1.G (VSS), DL2.G (VSS), DL3.G (VSS), DL4.G (VSS), DL5.G (VSS), DL6.G (VSS), DR1.G (VSS), DR2.G (VSS), DR3.G (VSS), DR4.G (VSS), DR5.G (VSS), DR6.G (VSS), J1.4 (Pin_4), J2.4 (Pin_4), J3.4 (Pin_4), J4.4 (Pin_4)
- net SCL: now also J1.2 (Pin_2), J2.2 (Pin_2), J3.2 (Pin_2), J4.2 (Pin_2)
- net SDA: now also J1.3 (Pin_3), J2.3 (Pin_3), J3.3 (Pin_3), J4.3 (Pin_3)
- net V2: now also C9.1
- net VB2: no longer C9.1
- net at U1.19 (GPIO14): now also DL1.I (In)
- net at U1.20 (GPIO15): now also DR1.I (In)
- new net: DR1.O (Out), DR2.I (In)
- new net: DR6.O (Out), J3.6 (Pin_6), J4.6 (Pin_6)
- new net: DL6.O (Out), J1.6 (Pin_6), J2.6 (Pin_6)
- new net: DR2.O (Out), DR3.I (In)
- new net: DR4.O (Out), DR5.I (In)
- new net: DR5.O (Out), DR6.I (In)
- new net: DL2.O (Out), DL3.I (In)
- new net: DL3.O (Out), DL4.I (In)
- new net: DR3.O (Out), DR4.I (In)
- new net: DL4.O (Out), DL5.I (In)
- new net: DL5.O (Out), DL6.I (In)
- new net: DL1.O (Out), DL2.I (In)
Other:
- moved on the sheet: D1, D10, D11, D12, D13, D14, D15, D16, D17, D18, D19, D2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

Commit message: PCB done for review
Parts:
- added C17, C18: 0.1uF, Capacitor_SMD:C_0603_1608Metric_Pad1.08x0.95mm_HandSolder, symbol Device:C
- added DL7, DL8, DL9, DR7, DR8, DR9: WS2812B_Unified, voltex_pico:WS2812B-4020_UP, symbol voltex_pico:WS2812B_Unified
- D1, D10, D11, D12, D13, D14, D15, D16, D17, D18, D19, D2, D20, D21, D3, D5, D6, D7, D8, D9: footprint voltex_pico:WS2812B-2835 -> voltex_pico:WS2812B-2835_EMBED
- DL5, DL6, DR5, DR6: footprint voltex_pico:WS2812B-4020 -> voltex_pico:WS2812B-4020_UP
Connections:
- net +3V3: no longer J1.1 (Pin_1), J2.1 (Pin_1), J3.1 (Pin_1), J4.1 (Pin_1)
- net +5V: now also C17.1, C18.1, DL7.V (VDD), DL8.V (VDD), DL9.V (VDD), DR7.V (VDD), DR8.V (VDD), DR9.V (VDD)
- net GND: now also C17.2, C18.2, DL7.G (VSS), DL8.G (VSS), DL9.G (VSS), DR7.G (VSS), DR8.G (VSS), DR9.G (VSS)
- net V1: now also J1.1 (Pin_1), J3.1 (Pin_1)
- net V2: now also J2.1 (Pin_1), J4.1 (Pin_1)
- net at DR4.O (Out), DR5.I (In): now also J2.6 (Pin_6), J4.6 (Pin_6)
- net at DL4.O (Out), DL5.I (In): now also J1.6 (Pin_6), J3.6 (Pin_6)
- new net: DR7.O (Out), DR8.I (In)
- new net: DR8.O (Out), DR9.I (In)
- new net: DL6.O (Out), DL7.I (In)
- new net: DL7.O (Out), DL8.I (In)
- new net: DR6.O (Out), DR7.I (In)
- new net: DL8.O (Out), DL9.I (In)
Other:
- moved on the sheet: C10, C11, C12, C13, C14, C15, C16, DL1, DL2, DL3, DL4, DL5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

Commit message: PCB v1.11
Parts:
- added C19, C20: 0.1uF, Capacitor_SMD:C_0603_1608Metric_Pad1.08x0.95mm_HandSolder, symbol Device:C
- added JP2: Bypass, Jumper:SolderJumper-2_P1.3mm_Open_RoundedPad1.0x1.5mm, symbol Jumper:SolderJumper_2_Open
- added U6: LM4040DBZ-3, voltex_pico:SOT-23-FAT, symbol Reference_Voltage:LM4040DBZ-3
- added U7: LP5907MFX-4.5, Package_TO_SOT_SMD:SOT-23-5, symbol Regulator_Linear:LP5907MFX-4.5
- added Z1: 3.3V, Diode_SMD:D_SOD-123F, symbol Device:D_Zener
- B1, B2, B3, B4, B5, B6: footprint voltex_pico:Choc_V1_HE -> voltex_pico:Choc_HE
- B7: footprint voltex_pico:Choc_V1_HE -> voltex_pico:Choc
- B8, B9: footprint voltex_pico:EVQP1K05M -> voltex_pico:SW_SKHHANA010
- JP1: value SolderJumper_2_Open -> Bypass
Connections:
- net +3V3: no longer JP1.1 (A)
- net +5V: now also JP1.1 (A)
- net GND: now also C19.2, C20.2, U6.2 (A), U7.2 (GND), Z1.2 (A)
- net Vref: now also C20.1, JP2.2 (B), U7.5 (OUT); no longer JP1.2 (B), U5.4 (Pin_4)
- net at R5.2, R6.2, U1.31 (GPIO26_ADC0)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: now also Z1.1 (K)
- net at U1.35 (ADC_VREF): now also U6.1 (K)
- new net Vboost: C19.1, JP1.2 (B), JP2.1 (A), U5.4 (Pin_4), U7.1 (IN), U7.3 (EN)
- no-connect marks 27 -> 26
Other:
- moved on the sheet: JP1, R5, U5

Commit message: PCB Pico v1.2 (remove unused parts)
Parts:
- removed JP1, JP2: Bypass, Jumper:SolderJumper-2_P1.3mm_Open_RoundedPad1.0x1.5mm, symbol Jumper:SolderJumper_2_Open
- removed U5: DC/DC, voltex_pico:DCDC_3to5, symbol Connector_Generic:Conn_02x02_Odd_Even
- U7: value LP5907MFX-4.5 -> LP5907MFX-4.2
Connections:
- net Vboost is gone; now on net VBUS: C19.1, U7.1 (IN), U7.3 (EN)
- net VBUS: now reaches U1.40 (VBUS), USB1.11 (VBUS), USB1.2 (VBUS)
- net +5V renamed VLED
Other:
- moved on the sheet: C19, C20, U7

Commit message: PCB v1.3 (use FPC)
Parts:
- J1, J2, J3, J4: footprint voltex_pico:Solder_6P -> voltex_pico:FPC6P1.0mm
Connections:
- net GND: now also J3.3 (Pin_3), J4.3 (Pin_3); no longer J3.4 (Pin_4), J4.4 (Pin_4)
- net SCL: now also J3.5 (Pin_5), J4.5 (Pin_5); no longer J3.2 (Pin_2), J4.2 (Pin_2)
- net SDA: now also J3.4 (Pin_4), J4.4 (Pin_4); no longer J3.3 (Pin_3), J4.3 (Pin_3)
- net V1: now also J3.6 (Pin_6); no longer J3.1 (Pin_1)
- net V2: now also J4.6 (Pin_6); no longer J4.1 (Pin_1)
- net VLED: now also J3.2 (Pin_2), J4.2 (Pin_2); no longer J3.5 (Pin_5), J4.5 (Pin_5)
- net at DL4.O (Out), DL5.I (In), J1.6 (Pin_6): now also J3.1 (Pin_1); no longer J3.6 (Pin_6)
- net at DR4.O (Out), DR5.I (In), J2.6 (Pin_6): now also J4.1 (Pin_1); no longer J4.6 (Pin_6)
Other:
- moved on the sheet: J3
Changed lines of the file:
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@@
 	)
 	(junction
-		(at 220.98 238.125)
-		(diameter 0)
-		(color 0 0 0 0)
-	)
-	(junction
 		(at 318.135 159.385)
 		(diameter 0)
@@
 	)
 	(junction
+		(at 220.345 238.125)
+		(diameter 0)
+		(color 0 0 0 0)
+	)
+	(junction
 		(at 127 160.02)
 		(diameter 0)
@@
 	(wire
 		(pts
-			(xy 219.71 248.285) (xy 224.79 248.285)
+			(xy 220.345 248.285) (xy 224.79 248.285)
 		)
 		(stroke
@@
 	(wire
 		(pts
-			(xy 220.98 238.125) (xy 229.87 238.125)
+			(xy 220.345 235.585) (xy 220.345 238.125)
 		)
 		(stroke
@@
 	(wire
 		(pts
+			(xy 220.345 238.125) (xy 229.87 238.125)
+		)
+		(stroke
+			(width 0)
+			(type default)
+		)
+	)
+	(wire
+		(pts
 			(xy 111.125 55.88) (xy 57.785 55.88)
 		)
@@
 	(wire
 		(pts
-			(xy 219.71 245.745) (xy 227.33 245.745)
+			(xy 220.345 245.745) (xy 227.33 245.745)
 		)
 		(stroke
@@
 	(wire
 		(pts
-			(xy 219.71 240.665) (xy 229.87 240.665)
+			(xy 220.345 240.665) (xy 229.87 240.665)
 		)
 		(stroke
@@
 	(wire
 		(pts
-			(xy 219.71 243.205) (xy 229.87 243.205)
+			(xy 220.345 243.205) (xy 229.87 243.205)
 		)
 		(stroke
@@
 	(wire
 		(pts
-			(xy 219.71 238.125) (xy 220.98 238.125)
-		)
-		(stroke
-			(width 0)
-			(type default)
-		)
-	)
-	(wire
-		(pts
 			(xy 342.9 186.69) (xy 342.9 189.23)
 		)
@@
 	(wire
 		(pts
-			(xy 219.71 250.825) (xy 220.345 250.825)
-		)
-		(stroke
-			(width 0)
-			(type default)
-		)
-	)
-	(wire
-		(pts
 			(xy 142.875 107.95) (xy 149.86 107.95)
 		)
@@
 	(wire
 		(pts
-			(xy 220.98 236.22) (xy 220.98 238.125)
-		)
-		(stroke
-			(width 0)
-			(type default)
-		)
-	)
-	(wire
-		(pts
 			(xy 72.39 209.55) (xy 87.63 209.55)
 		)
@@
 	)
 	(label "V1"
-		(at 220.98 236.22 0)
+		(at 220.345 235.585 0)
 		(effects
 			(font
@@
 	(symbol
 		(lib_id "Connector:Conn_01x06_Socket")
-		(at 214.63 243.205 0)
-		(mirror y)
+		(at 215.265 245.745 180)
 		(unit 1)
 		(exclude_from_sim no)
@@
 		(dnp no)
 		(property "Reference" "J3"
-			(at 212.725 236.855 0)
+			(at 213.36 252.095 0)
 			(effects
 				(font
@@
 		)
 		(property "Value" "Conn_01x06_Socket"
-			(at 212.725 245.7449 0)
+			(at 213.36 243.2051 0)
 			(effects
 				(font
@@
 			)
 		)
-		(property "Footprint" "voltex_pico:Solder_6P"
-			(at 214.63 243.205 0)
+		(property "Footprint" "voltex_pico:FPC6P1.0mm"
+			(at 215.265 245.745 0)
 			(effects
 				(font
@@
 		)
 		(property "Datasheet" "~"
-			(at 214.63 243.205 0)
+			(at 215.265 245.745 0)
 			(effects
 				(font
@@
 		)
 		(property "Description" "Generic connector, single row, 01x06, script generated"
-			(at 214.63 243.205 0)
+			(at 215.265 245.745 0)
 			(effects
 				(font
@@
 			)
 		)
-		(property "Footprint" "voltex_pico:Solder_6P"
+		(property "Footprint" "voltex_pico:FPC6P1.0mm"
 			(at 234.95 243.205 0)
 			(effects
@@
 			)
 		)
-		(property "Footprint" "voltex_pico:Solder_6P"
+		(property "Footprint" "voltex_pico:FPC6P1.0mm"
 			(at 250.825 243.205 0)
 			(effects
@@
 	(symbol
 		(lib_id "Connector:Conn_01x06_Socket")
-		(at 270.51 243.205 0)
+		(at 270.51 245.745 0)
+		(mirror x)
 		(unit 1)
 		(exclude_from_sim no)
@@
 		(dnp no)
 		(property "Reference" "J4"
-			(at 272.415 236.855 0)
+			(at 272.415 252.095 0)
 			(effects
 				(font
@@
 		)
 		(property "Value" "Conn_01x06_Socket"
-			(at 272.415 245.7449 0)
+			(at 272.415 243.2051 0)
 			(effects
 				(font
@@
 			)
 		)
-		(property "Footprint" "voltex_pico:Solder_6P"
-			(at 270.51 243.205 0)
+		(property "Footprint" "voltex_pico:FPC6P1.0mm"
+			(at 270.51 245.745 0)
 			(effects
 				(font
@@
 		)
 		(property "Datasheet" "~"
-			(at 270.51 243.205 0)
+			(at 270.51 245.745 0)
 			(effects
 				(font
@@
 		)
 		(property "Description" "Generic connector, single row, 01x06, script generated"
-			(at 270.51 243.205 0)
+			(at 270.51 245.745 0)
 			(effects
 				(font
