File: PCB/pico/voltex_pico.kicad_pcb (KiCad board)
At the start: 2 copper layers, 274.8 x 152.8 mm, 63 parts, among them U1 PiPico, U2 ADG708BRUZ, U3 TMAG5273, U4 TMAG5273, U5 DC/DC

Commit message: PCB progress 70%
Parts:
- removed C26: 0.1uF, Capacitor_SMD:C_0603_1608Metric_Pad1.08x0.95mm_HandSolder
- removed JA1, JA2, JB1, JB2: Conn_01x04, voltex_pico:SH1.0_4P_Solder_Combo
- added C12: 0.1uF, Capacitor_SMD:C_0603_1608Metric_Pad1.08x0.95mm_HandSolder, B.Cu at (251.6, 134.0)
- added C13: 0.1uF, Capacitor_SMD:C_0603_1608Metric_Pad1.08x0.95mm_HandSolder, B.Cu at (314.5, 134.0)
- added C14: 0.1uF, Capacitor_SMD:C_0603_1608Metric_Pad1.08x0.95mm_HandSolder, B.Cu at (165.1, 204.0)
- added C15: 0.1uF, Capacitor_SMD:C_0603_1608Metric_Pad1.08x0.95mm_HandSolder, B.Cu at (266.2, 203.4)
- added C16: 0.1uF, Capacitor_SMD:C_0603_1608Metric_Pad1.08x0.95mm_HandSolder, B.Cu at (226.6, 93.0)
- added C8: 0.1uF, Capacitor_SMD:C_0603_1608Metric_Pad1.08x0.95mm_HandSolder, F.Cu at (150.2, 118.1)
- added C9: 0.1uF, Capacitor_SMD:C_0603_1608Metric_Pad1.08x0.95mm_HandSolder, F.Cu at (278.2, 118.1)
- added DL1: WS2812B_Unified, voltex_pico:WS2812B-4020, F.Cu at (126.2, 222.1)
- added DL2: WS2812B_Unified, voltex_pico:WS2812B-4020, F.Cu at (112.2, 204.1)
- added DL3: WS2812B_Unified, voltex_pico:WS2812B-4020, F.Cu at (96.2, 188.1)
- added DL4: WS2812B_Unified, voltex_pico:WS2812B-4020, F.Cu at (84.2, 171.1)
- added DL5: WS2812B_Unified, voltex_pico:WS2812B-4020, F.Cu at (84.2, 155.1)
- added DL6: WS2812B_Unified, voltex_pico:WS2812B-4020, F.Cu at (84.2, 139.1)
- added DR1: WS2812B_Unified, voltex_pico:WS2812B-4020, F.Cu at (302.2, 222.1)
- added DR2: WS2812B_Unified, voltex_pico:WS2812B-4020, F.Cu at (316.2, 204.1)
- added DR3: WS2812B_Unified, voltex_pico:WS2812B-4020, F.Cu at (332.2, 188.1)
- added DR4: WS2812B_Unified, voltex_pico:WS2812B-4020, F.Cu at (344.2, 171.1)
- added DR5: WS2812B_Unified, voltex_pico:WS2812B-4020, F.Cu at (344.2, 155.1)
- added DR6: WS2812B_Unified, voltex_pico:WS2812B-4020, F.Cu at (344.2, 139.1)
- added J1: Conn_01x06_Socket, voltex_pico:Solder_6P, F.Cu at (94.2, 115.1)
- added J2: Conn_01x06_Socket, voltex_pico:Solder_6P, F.Cu at (334.2, 115.1)
- added J3: Conn_01x06_Socket, voltex_pico:Solder_6P, F.Cu at (150.2, 101.1)
- added J4: Conn_01x06_Socket, voltex_pico:Solder_6P, F.Cu at (278.2, 101.1)
- C10, C11: moved to B.Cu
- moved C11 74.3 mm to (196.5, 140.7)
- moved C10 42.1 mm to (125.5, 134.0)
- moved U3 6.53 mm to (150.2, 115.1)
- moved U4 4.80 mm to (278.2, 115.1)
Connections:
- C10 pad 1: /VB1 -> +5V
- C11 pad 1: /VB2 -> +5V
- U1 pad 19: unconnected-(U1-GPIO14-Pad19) -> Net-(DL1-In)
- U1 pad 20: unconnected-(U1-GPIO15-Pad20) -> Net-(DR1-In)
Routing:
- net +5V: track 331.7 -> 1732.3 mm, vias 0 -> 11
- net /K8: track 0.00 -> 150.1 mm, vias 0 -> 2
- net /K9: track 0.00 -> 127.3 mm, vias 0 -> 2
- net /K7: track 0.00 -> 125.4 mm, vias 0 -> 1
- net Net-(DR1-In): track 0.00 -> 104.8 mm, vias 0 -> 2
- net Net-(DL1-In): track 0.00 -> 89.0 mm
- net GND: track 0.00 -> 45.9 mm, vias 0 -> 30
- net Net-(DL3-Out): track 0.00 -> 30.1 mm
- net Net-(DR1-Out): track 0.00 -> 29.9 mm
- net Net-(DL1-Out): track 0.00 -> 29.6 mm
- net Net-(DL2-Out): track 0.00 -> 28.1 mm
- net Net-(DR3-Out): track 0.00 -> 24.0 mm
- net Net-(DR2-Out): track 0.00 -> 23.9 mm
- net Net-(DL5-Out): track 0.00 -> 22.4 mm
- net Net-(DL4-Out): track 0.00 -> 22.1 mm
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- added copper zone on B.Cu, net GND
- added copper zone on F.Cu, net GND

Commit message: PCB done for review
Parts:
- added C17: 0.1uF, Capacitor_SMD:C_0603_1608Metric_Pad1.08x0.95mm_HandSolder, F.Cu at (162.4, 112.4)
- added C18: 0.1uF, Capacitor_SMD:C_0603_1608Metric_Pad1.08x0.95mm_HandSolder, F.Cu at (282.4, 112.4)
- added DL7: WS2812B_Unified, voltex_pico:WS2812B-4020_UP, F.Cu at (154.2, 110.9)
- added DL8: WS2812B_Unified, voltex_pico:WS2812B-4020_UP, F.Cu at (148.0, 109.3)
- added DL9: WS2812B_Unified, voltex_pico:WS2812B-4020_UP, F.Cu at (143.4, 104.7)
- added DR7: WS2812B_Unified, voltex_pico:WS2812B-4020_UP, F.Cu at (274.2, 110.9)
- added DR8: WS2812B_Unified, voltex_pico:WS2812B-4020_UP, F.Cu at (268.0, 109.3)
- added DR9: WS2812B_Unified, voltex_pico:WS2812B-4020_UP, F.Cu at (263.4, 104.7)
- D1, D10, D11, D12, D13, D14, D15, D16, D17, D18, D19, D2, D20, D21, D3, D5, D6, D7, D8, D9: footprint voltex_pico:WS2812B-2835 -> voltex_pico:WS2812B-2835_EMBED; moved to B.Cu
- DL5, DL6, DR5, DR6: footprint voltex_pico:WS2812B-4020 -> voltex_pico:WS2812B-4020_UP
- moved DL5 95.2 mm to (165.0, 104.7), turned to 60 degrees
- moved DL6 81.8 mm to (160.4, 109.3), turned to 30 degrees
- moved DR5 77.7 mm to (285.0, 104.7), turned to 60 degrees
- moved DR6 70.4 mm to (280.4, 109.3), turned to 30 degrees
- moved JP1 35.0 mm to (238.2, 193.1), turned to -90 degrees
- moved U5 34.7 mm to (239.2, 193.1), turned to -90 degrees
- moved C14 24.9 mm to (140.2, 202.3), turned to 180 degrees
- moved C8 23.0 mm to (154.2, 95.5), turned to 0 degrees
- moved C9 23.0 mm to (274.2, 95.5), turned to 0 degrees
- moved C15 22.0 mm to (288.2, 202.3)
- moved C11 21.1 mm to (177.2, 132.1)
- moved U3 17.1 mm to (154.2, 98.5), turned to 180 degrees
- moved U4 17.1 mm to (274.2, 98.5), turned to 180 degrees
- moved J3 14.6 mm to (154.2, 115.1), turned to 90 degrees
- moved J4 14.6 mm to (274.2, 115.1), turned to 90 degrees
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Connections:
- J1 pad 1: +3V3 -> /V1
- J1 pad 6: (no net) -> Net-(DL4-Out)
- J2 pad 1: +3V3 -> /V2
- J2 pad 6: (no net) -> Net-(DR4-Out)
- J3 pad 1: +3V3 -> /V1
- J3 pad 6: (no net) -> Net-(DL4-Out)
- J4 pad 1: +3V3 -> /V2
- J4 pad 6: (no net) -> Net-(DR4-Out)
Routing:
- net /SCL: track 1.89 -> 405.9 mm, vias 1 -> 7
- net /SDA: track 1.89 -> 389.2 mm, vias 1 -> 5
- net GND: track 45.9 -> 238.1 mm, vias 30 -> 90
- net Net-(DL4-Out): track 22.1 -> 166.4 mm, vias 0 -> 1
- net Net-(DR4-Out): track 17.4 -> 146.5 mm, vias 0 -> 1
- net /V2: track 230.9 -> 357.8 mm, vias 1 -> 4
- net /V1: track 204.6 -> 308.0 mm, vias 1 -> 2
- net +5V: track 1732.3 -> 1793.2 mm, vias 11 -> 26
- net Net-(D12-In): track 119.3 -> 144.8 mm
- net Net-(DR1-In): track 104.8 -> 130.0 mm
- net Net-(DL1-In): track 89.0 -> 110.1 mm
- net Net-(D18-In): track 122.2 -> 143.3 mm, vias 2 -> 0
- net Net-(D21-In): track 142.0 -> 159.0 mm, vias 0 -> 2
- net Net-(DL5-Out): track 22.4 -> 7.13 mm
- net Net-(D1-Out): track 145.5 -> 132.1 mm
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Other:
- board size 274.8 x 152.8 mm -> 275 x 153 mm
- board text added: "Voltex Pico"
- board text added: "v1.0"

Commit message: PCB v1.0
Routing:
- net /K1: track 57.2 -> 87.1 mm
- net Net-(D21-In): track 159.0 -> 166.6 mm
- net Vref: track 593.7 -> 587.2 mm
- net /S5: track 78.1 -> 72.4 mm
- net /K6: track 92.7 -> 97.7 mm
- net Net-(D1-Out): track 132.1 -> 128.8 mm
- net /V2: track 357.8 -> 355.0 mm
- net Net-(DR1-In): track 130.0 -> 127.8 mm
- net +5V: track 1793.2 -> 1791.8 mm
- net GND: vias 90 -> 96
Other:
- outline, holes or cut-outs redrawn

Commit message: PCB v1.11
Parts:
- added C19: 0.1uF, Capacitor_SMD:C_0603_1608Metric_Pad1.08x0.95mm_HandSolder, B.Cu at (234.5, 198.9)
- added C20: 0.1uF, Capacitor_SMD:C_0603_1608Metric_Pad1.08x0.95mm_HandSolder, B.Cu at (234.5, 192.9)
- added JP2: Bypass, Jumper:SolderJumper-2_P1.3mm_Open_RoundedPad1.0x1.5mm, B.Cu at (237.8, 195.9)
- added U6: LM4040DBZ-3, voltex_pico:SOT-23-FAT, B.Cu at (222.9, 187.8)
- added U7: LP5907MFX-4.5, Package_TO_SOT_SMD:SOT-23-5, B.Cu at (234.4, 195.9)
- added Z1: 3.3V, Diode_SMD:D_SOD-123F, B.Cu at (214.7, 193.4)
- B1, B2, B3, B4, B5, B6: footprint voltex_pico:Choc_V1_HE -> voltex_pico:Choc_HE
- B7: footprint voltex_pico:Choc_V1_HE -> voltex_pico:Choc
- B8, B9: footprint voltex_pico:EVQP1K05M -> voltex_pico:SW_SKHHANA010
- JP1: value SolderJumper_2_Open -> Bypass
- moved R1 4.00 mm to (202.4, 86.9)
- moved R2 4.00 mm to (225.9, 87.0)
- moved C7 2.05 mm to (221.6, 183.4)
- moved C5 1.10 mm to (146.0, 205.0)
- moved C6 1.10 mm to (272.0, 205.0)
- moved C2 1.10 mm to (177.5, 142.3)
- moved C3 1.10 mm to (240.5, 142.3)
- moved C4 1.10 mm to (303.5, 142.3)
- moved C1 1.10 mm to (114.5, 142.3)
- moved C16 1.00 mm to (225.6, 93.0)
- moved R3 0.71 mm to (206.7, 173.0)
- moved R4 0.64 mm to (206.7, 171.3)
Connections:
- JP1 pad 1: +3V3 -> +5V
- JP1 pad 2: Vref -> Vboost
- U1 pad 35: unconnected-(U1-ADC_VREF-Pad35) -> Net-(U1-ADC_VREF)
- U5 pad 4: Vref -> Vboost
Routing:
- net Vref: track 587.2 -> 620.7 mm, vias 7 -> 6
- net Vboost: track 0.00 -> 25.2 mm, vias 0 -> 2
- net +3V3: track 48.7 -> 37.7 mm
- net /S5: track 72.4 -> 82.9 mm
- net /S1: track 79.0 -> 86.7 mm
- net /K5: track 128.0 -> 134.9 mm
- net Net-(D1-In): track 106.0 -> 112.5 mm
- net GND: track 238.1 -> 243.6 mm, vias 96 -> 112
- net +5V: track 1791.8 -> 1796.9 mm
- net /S6: track 113.0 -> 118.0 mm
- net /K4: track 81.3 -> 85.8 mm
- net Net-(USB1-CC2): track 7.97 -> 12.0 mm
- net Net-(USB1-CC1): track 8.63 -> 12.6 mm
- net /K6: track 97.7 -> 101.6 mm
- net Net-(D15-In): track 137.3 -> 140.8 mm
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Other:
- outline, holes or cut-outs redrawn
- board text added: "v1.11"
- board text removed: "v1.0"

Commit message: PCB Pico v1.2 (remove unused parts)
Parts:
- removed JP1, JP2: Bypass, Jumper:SolderJumper-2_P1.3mm_Open_RoundedPad1.0x1.5mm
- removed U5: DC/DC, voltex_pico:DCDC_3to5
- U7: value LP5907MFX-4.5 -> LP5907MFX-4.2
Connections:
- net +5V renamed VLED
- C19 pad 1: Vboost -> VBUS
- U1 pad 40: Net-(U1-VBUS) -> VBUS
- U7 pad 1: Vboost -> VBUS
- U7 pad 3: Vboost -> VBUS
- USB1 pad 11: Net-(U1-VBUS) -> VBUS
- USB1 pad 2: Net-(U1-VBUS) -> VBUS
Routing:
- net VBUS: track 0.00 -> 163.7 mm, vias 0 -> 6
- net Net-(U1-VBUS): track 116.5 -> 0.00 mm, vias 3 -> 0
- net Vboost: track 25.2 -> 0.00 mm, vias 2 -> 0
- net +3V3: track 37.7 -> 22.7 mm, vias 3 -> 1
- net Vref: track 620.7 -> 611.5 mm
- net VLED: track 1796.9 -> 1789.0 mm
- net /S6: track 118.0 -> 115.2 mm
- net /K5: track 134.9 -> 132.0 mm
- net /K6: track 101.6 -> 104.1 mm
- net /S5: track 82.9 -> 80.5 mm
- net Net-(U1-GPIO21): track 28.5 -> 29.5 mm
- net GND: vias 112 -> 119
Other:
- board text added: "v1.2"
- board text removed: "v1.11"

Commit message: PCB v1.3 (use FPC)
Parts:
- J1, J2, J3, J4: footprint voltex_pico:Solder_6P -> voltex_pico:FPC6P1.0mm
- moved J3 1.80 mm to (154.2, 116.9), turned to 0 degrees
- moved J4 1.80 mm to (274.2, 116.9), turned to 0 degrees
- turned J1 to -135 degrees
- turned J2 to 135 degrees
Connections:
- J3 pad 1: /V1 -> Net-(DL4-Out)
- J3 pad 2: /SCL -> VLED
- J3 pad 3: /SDA -> GND
- J3 pad 4: GND -> /SDA
- J3 pad 5: VLED -> /SCL
- J3 pad 6: Net-(DL4-Out) -> /V1
- J4 pad 1: /V2 -> Net-(DR4-Out)
- J4 pad 2: /SCL -> VLED
- J4 pad 3: /SDA -> GND
- J4 pad 4: GND -> /SDA
- J4 pad 5: VLED -> /SCL
- J4 pad 6: Net-(DR4-Out) -> /V2
Routing:
- net GND: track 243.6 -> 246.4 mm, vias 119 -> 121
- net VLED: track 1789.0 -> 1791.9 mm, vias 26 -> 30
- net Net-(DL4-Out): track 166.4 -> 169.1 mm, vias 1 -> 2
- net /V1: track 308.0 -> 310.7 mm, vias 2 -> 4
- net /SDA: track 388.9 -> 390.3 mm, vias 5 -> 7
- net Net-(DR6-Out): track 8.13 -> 6.81 mm
- net Net-(DL6-Out): track 8.24 -> 6.96 mm
- net /SCL: track 405.6 -> 406.7 mm, vias 7 -> 9
- net /V2: track 355.0 -> 355.4 mm, vias 4 -> 6
- net Net-(DR4-Out): track 146.7 -> 146.8 mm, vias 1 -> 2
Other:
- board text added: "github.com/whowechina"
- board text added: "v1.3"
- board text removed: "v1.2"

Commit message: PCB v1.31 (FPC alignment)
Parts:
- moved J1 0.78 mm to (95.6, 117.6)
- moved J2 0.78 mm to (332.8, 117.6)
Routing:
- net VLED: track 1791.9 -> 1790.3 mm
- net Net-(DR4-Out): track 146.8 -> 145.6 mm
- net /SCL: track 406.7 -> 407.4 mm
- net /SDA: track 390.3 -> 391.0 mm
Other:
- board text added: "v1.31"
- board text removed: "v1.3"
