File: PCB/jumbo/voltex_jumbo.kicad_sch (KiCad schematic)
At the start: 83 parts, among them U1 PiPico, U2 ADG708BRUZ, U3 TMAG5273, U4 TMAG5273, U6 LM4040DBZ-3, U7 LP5907MFX-4.2

Commit message: Jumbo PCB continued
Parts:
- removed C1, C2, C3, C4, C7: 0.1uF, Capacitor_SMD:C_0603_1608Metric_Pad1.08x0.95mm_HandSolder, symbol Device:C
- C6: Side (none) -> R
- U1: footprint voltex_jumbo:RPi_Pico_SMD_Pins -> voltex_jumbo:RPi_Pico_SMD_No_SWD
- renumbered B8 to B5, C19 to C1, C20 to C2, C8 to C3, C9 to C4
Connections:
- net GND: no longer C6.2
- net Gref: now also C6.2
- net K5R: now also JR2.2 (Pin_2); no longer JR2.3 (Pin_3)
- net K6R: now also JR2.3 (Pin_3); no longer JR2.2 (Pin_2)
- net S5R: now also JR1.3 (Pin_3); no longer JR1.2 (Pin_2)
- net S6R: now also JR1.2 (Pin_2); no longer JR1.3 (Pin_3)
- net D-: now reaches U1.TP2 (USB1), USB1.5 (DN2), USB1.7 (DN1)
- net D+: now reaches U1.TP3 (USB2), USB1.6 (DP1), USB1.8 (DP2)
- net K4 renamed S4_K4
- net K5 renamed S5_K6
- net S5_K6: now also U1.7 (GPIO5); no longer U1.9 (GPIO6)
- net K6 renamed S6_K5
- net S6_K5: now also U1.9 (GPIO6); no longer U1.7 (GPIO5)
- no-connect marks 29 -> 26
Other:
- moved on the sheet: C10, C11, C12, C13, C14, C15, C16, C17, C18, C3, C4

Commit message: Jumbo PCB v1.0
Parts:
- removed JR2: BT, voltex_jumbo:SH1.0_4P_Solder_Combo, symbol Connector:Conn_01x04_Socket
- added C13, C14, C15: 0.1uF, Capacitor_SMD:C_0603_1608Metric_Pad1.08x0.95mm_HandSolder, symbol Device:C
- added JL2: BT, voltex_jumbo:SH1.0_4P_Solder_Combo, symbol Connector_Generic:Conn_01x04
- C16, C17, C18, C4: Side (none) -> R
- JL1: value BT_Hall -> Hall
- JR1: value HALL -> HALL_BT
- R5: value 2K -> 1K
- R6: value 10K -> 50K
- U6: value LM4040DBZ-3 -> LM4040DBZ-2.1
- renumbered C13 to C10, C14 to C11, C15 to C12, C10 to C7, C11 to C8, C12 to C9, JL2 to JL3, JL3 to JL4, JL4 to JL5
Connections:
- net S4R is gone; now on net S4_K4_R: H3.2 (OUT), JR1.1 (Pin_1)
- net S5R is gone; now on net S5_K6_R: H6.2 (OUT), JR1.3 (Pin_3)
- net S6R is gone; now on net S6_K5_R: H4.2 (OUT), JR1.2 (Pin_2)
- net GND: now also C13.2, C14.2, C15.2, JL2.4 (Pin_4)
- net VLED: now also C13.1, C14.1, C15.1
- net K4R renamed S4_K4_R
- net K5R renamed S6_K5_R
- net K6R renamed S5_K6_R
- net S4_K4 renamed S4
- net S4: no longer U1.10 (GPIO7)
- removed net S5_K6: JL1.3 (Pin_3), U1.7 (GPIO5), U2.11 (S6)
- removed net S6_K5: JL1.2 (Pin_2), U1.9 (GPIO6), U2.12 (S5)
- new net K4: JL2.1 (Pin_1), U1.10 (GPIO7)
- new net K5: JL2.2 (Pin_2), U1.9 (GPIO6)
- new net K6: JL2.3 (Pin_3), U1.7 (GPIO5)
- new net S5: JL1.3 (Pin_3), U2.12 (S5)
- new net S6: JL1.2 (Pin_2), U2.11 (S6)
- no-connect marks 26 -> 29
Other:
- note added: "Hall and BT Shared"
- note removed: "Shared Connector"
- moved on the sheet: JL3, JL4, JL5
