File: PCB/jumbo/voltex_jumbo.kicad_pcb (KiCad board)
At the start: 2 copper layers, 195.9 x 212.8 mm, 83 parts, among them U1 PiPico, U2 ADG708BRUZ, U3 TMAG5273, U4 TMAG5273, U6 LM4040DBZ-3, U7 LP5907MFX-4.2

Commit message: Jumbo PCB continued
Parts:
- removed the C1 at (153.5, 135.3)
- removed the C2 at (230.5, 135.3)
- removed C7: 0.1uF, Capacitor_SMD:C_0603_1608Metric_Pad1.08x0.95mm_HandSolder
- C3: renamed from C8; moved to B.Cu
- C4: renamed from C9; moved to F.Cu
- D4, JR1, JR2, JR3, JR4, JR5, U3: moved to B.Cu
- JL1, JL2, JL3, JL4, U4: moved to F.Cu
- U1: footprint voltex_jumbo:RPi_Pico_SMD_Pins -> voltex_jumbo:RPi_Pico_SMD_No_SWD
- moved C6 140.7 mm to (233.9, 113.1)
- moved C1 106.8 mm to (202.1, 97.1), turned to 0 degrees
- moved U7 101.1 mm to (202.2, 100.1), turned to -90 degrees
- moved C5 101.0 mm to (198.8, 112.1), turned to 0 degrees
- moved R5 95.6 mm to (194.6, 96.4)
- moved R6 95.6 mm to (194.6, 98.0)
- moved Z1 95.6 mm to (194.1, 100.1)
- moved C2 95.5 mm to (202.1, 103.1), turned to 0 degrees
- moved U2 89.5 mm to (186.2, 98.1), turned to -90 degrees
- moved U6 83.4 mm to (203.0, 106.7), turned to 90 degrees
- moved R3 82.9 mm to (214.9, 90.5), turned to 0 degrees
- moved R4 79.7 mm to (214.8, 92.1), turned to 0 degrees
- moved JR1 46.0 mm to (239.2, 106.1), turned to -90 degrees
- moved JL1 44.0 mm to (239.2, 106.1), turned to 90 degrees
- moved JL4 44.0 mm to (239.2, 66.1), turned to 90 degrees
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- renumbered B8 to B5, C19 to C1, C20 to C2
Connections:
- net /K4 renamed /S4_K4
- net Net-(U1-USB1) renamed /D-
- net Net-(U1-USB2) renamed /D+
- C6 pad 2: GND -> Gref
- JL1 pad 2: /K6 -> /S6_K5
- JL1 pad 3: /K5 -> /S5_K6
- JR1 pad 2: /S5R -> /S6R
- JR1 pad 3: /S6R -> /S5R
- JR2 pad 2: /K6R -> /K5R
- JR2 pad 3: /K5R -> /K6R
- U1 pad 7: /K6 -> /S5_K6
- U1 pad 9: /K5 -> /S6_K5
- U2 pad 11: /K5 -> /S5_K6
- U2 pad 12: /K6 -> /S6_K5
Routing:
- net VLED: track 0.00 -> 1138.0 mm, vias 0 -> 14
- net Vref: track 0.00 -> 282.6 mm, vias 0 -> 9
- net Gref: track 0.00 -> 249.5 mm, vias 0 -> 4
- net /LED_BT: track 0.00 -> 218.6 mm, vias 0 -> 2
- net /SDA: track 0.00 -> 196.5 mm, vias 0 -> 4
- net /SCL: track 0.00 -> 195.1 mm, vias 0 -> 3
- net /K1: track 0.00 -> 194.7 mm
- net /LED_L: track 0.00 -> 169.6 mm
- net /V2: track 0.00 -> 167.8 mm, vias 0 -> 4
- net /LED_R: track 0.00 -> 164.7 mm, vias 0 -> 1
- net /K6R: track 0.00 -> 151.4 mm, vias 0 -> 2
- net /S1: track 0.00 -> 147.6 mm, vias 0 -> 2
- net /S5R: track 0.00 -> 145.6 mm, vias 0 -> 1
- net Net-(DL4-Out): track 0.00 -> 130.4 mm
- net /S3: track 0.00 -> 122.4 mm, vias 0 -> 2
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
Commit message: Jumbo PCB v1.0
Parts:
- removed the C3 at (99.7, 99.2)
- removed the C4 at (86.0, 117.8)
- removed JR2: BT, voltex_jumbo:SH1.0_4P_Solder_Combo
- added C7: 0.1uF, Capacitor_SMD:C_0603_1608Metric_Pad1.08x0.95mm_HandSolder, B.Cu at (174.7, 123.2)
- added C8: 0.1uF, Capacitor_SMD:C_0603_1608Metric_Pad1.08x0.95mm_HandSolder, B.Cu at (223.0, 134.7)
- added C9: 0.1uF, Capacitor_SMD:C_0603_1608Metric_Pad1.08x0.95mm_HandSolder, B.Cu at (187.6, 224.3)
- added JL2: BT, voltex_jumbo:SH1.0_4P_Solder_Combo, F.Cu at (239.2, 96.1)
- C10, C11, C13, C14, C15, C18: moved to F.Cu
- C17: moved to B.Cu
- JL1: value BT_Hall -> Hall
- JR1: value HALL -> HALL_BT
- R5: value 2K -> 1K
- R6: value 10K -> 50K
- U6: value LM4040DBZ-3 -> LM4040DBZ-2.1
- moved C18 177.4 mm to (254.4, 43.5), turned to 0 degrees
- moved C11 162.8 mm to (90.8, 77.1), turned to 180 degrees
- moved C12 161.5 mm to (254.4, 43.5)
- moved C16 156.0 mm to (157.3, 212.5)
- moved C13 139.7 mm to (219.7, 147.2), turned to 180 degrees
- moved C15 110.3 mm to (206.3, 208.6)
- moved C10 99.5 mm to (149.3, 213.0)
- moved C14 67.0 mm to (142.7, 147.2)
- moved C17 16.7 mm to (102.8, 63.4)
- moved JL3 10.0 mm to (239.2, 86.1)
- moved C6 5.00 mm to (233.9, 118.1)
- moved B5 2.00 mm to (232.2, 53.1)
- renumbered D8 to D1, D2 to D10, D10 to D2, D1 to D8, JL2 to JL3, JL3 to JL4, JL4 to JL5
Connections:
- B1 pad 3: /K5R -> /S6_K5_R
- B2 pad 3: /K4R -> /S4_K4_R
- B3 pad 3: /K6R -> /S5_K6_R
- D1 pad O: unconnected-(D8-Out-PadO) -> Net-(D1-Out)
- D1 pad OB: unconnected-(D8-OutB-PadOB) -> Net-(D1-OutB)
- D10 pad O: Net-(D12-In) -> unconnected-(D10-Out-PadO)
- D10 pad OB: Net-(D1-InB) -> unconnected-(D10-OutB-PadOB)
- D2 pad O: unconnected-(D10-Out-PadO) -> Net-(D12-In)
- D2 pad OB: unconnected-(D10-OutB-PadOB) -> Net-(D1-InB)
- D8 pad O: Net-(D1-Out) -> unconnected-(D8-Out-PadO)
- D8 pad OB: Net-(D1-OutB) -> unconnected-(D8-OutB-PadOB)
- H3 pad 2: /S4R -> /S4_K4_R
- H4 pad 2: /S6R -> /S6_K5_R
- H6 pad 2: /S5R -> /S5_K6_R
- JL1 pad 1: /S4_K4 -> /S4
- JL1 pad 2: /S6_K5 -> /S6
- JL1 pad 3: /S5_K6 -> /S5
- JR1 pad 1: /S4R -> /S4_K4_R
- JR1 pad 2: /S6R -> /S6_K5_R
- JR1 pad 3: /S5R -> /S5_K6_R
- U1 pad 10: /S4_K4 -> /K4
- U1 pad 7: /S5_K6 -> /K6
- U1 pad 9: /S6_K5 -> /K5
- U2 pad 11: /S5_K6 -> /S6
- U2 pad 12: /S6_K5 -> /S5
- U2 pad 7: /S4_K4 -> /S4
Routing:
- net Net-(D1-OutB): track 0.00 -> 209.7 mm, vias 0 -> 2
- net /K6R: track 151.4 -> 0.00 mm, vias 2 -> 0
- net /S5_K6_R: track 0.00 -> 149.6 mm, vias 0 -> 1
- net /S5R: track 145.6 -> 0.00 mm, vias 1 -> 0
- net /S6_K5_R: track 0.00 -> 116.4 mm, vias 0 -> 3
- net /K5R: track 110.3 -> 0.00 mm, vias 2 -> 0
- net /S6R: track 109.9 -> 0.00 mm, vias 3 -> 0
- net /LED_BT_R: track 86.3 -> 193.2 mm, vias 0 -> 2
- net /K4R: track 102.4 -> 0.00 mm, vias 2 -> 0
- net Net-(D3-Out): track 0.00 -> 96.5 mm, vias 0 -> 2
- net /KX: track 3.41 -> 87.3 mm, vias 0 -> 4
- net /LED_R: track 164.7 -> 247.3 mm, vias 1 -> 5
- net Net-(D1-InB): track 32.3 -> 113.4 mm, vias 0 -> 2
- net /S6_K5: track 77.1 -> 0.00 mm, vias 1 -> 0
- net Net-(D1-Out): track 79.3 -> 155.9 mm, vias 4 -> 6
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- added copper zone on B.Cu, net GND
- added copper zone on F.Cu, net GND
Other:
- board text added: "R"

Commit message: Jumbo PCB v1.01 (silkscreen fix)
Other:
- outline, holes or cut-outs redrawn
- board text added: "v1.01"
- board text removed: "v1.0"
